File: Protoboard/Protoboard-Araceli/Protoboard-Araceli.kicad_sch (KiCad schematic)
At the start: 24 parts, among them SW1 SW_DIP_x04, SW3 SW_Push, U1 PIC18F4550-IP, U2 HDSP-7803, U3 HDSP-7803

Commit message: Araceli aded
Parts:
- removed U3: HDSP-7803, Display_7Segment:HDSP-7801, symbol Display_Character:HDSP-7803
Connections:
- net +5V: now also U1.11 (VDD)
- net GND: now also SW1.5, SW1.6, SW1.7, SW1.8, U1.12 (VSS)
- net at BAR1.8 (A), R3.1: now also U2.8 (C)
- net at BAR1.6 (A), R5.1: now also U2.4 (E); no longer U2.5 (D)
- net at SW1.3: now also U2.6 (CC)
- net at SW1.4: now also BAR1.11 (K), BAR1.12 (K), BAR1.13 (K), BAR1.14 (K), BAR1.15 (K), BAR1.16 (K), BAR1.17 (K), BAR1.18 (K), BAR1.19 (K), BAR1.20 (K)
- net at BAR1.10 (A), R1.1: now also U2.10 (A); no longer U2.7 (DP)
- net at BAR1.3 (A), R8.1: now also U2.7 (DP)
- net at BAR1.4 (A), R7.1: now also U2.3 (G)
- net at BAR1.5 (A), R6.1: now also U2.2 (F); no longer U2.8 (C)
- net at BAR1.7 (A), R4.1: now also U2.5 (D); no longer U2.4 (E)
- net at BAR1.9 (A), R2.1: now also U2.9 (B)
Other:
- title: (none) -> Protoboard Araceli
- moved on the sheet: BAR1, R1, R11, R18, R19, SW, SW1, SW3, U1, U2
