File: Protoboard/Protoboard-Alejandra/Protoboard-Alejandra.kicad_sch (KiCad schematic)
At the start: 22 parts, among them SW1 SW_DIP_x08, SW2 SW_Push, U1 PIC18LF4550-IP

Commit message: Protoboard alejandra finish
Parts:
- added R19: 470, symbol Device:R
- added R20: 10K, symbol Device:R
Connections:
- net +5V: now also R20.2
- net GND: now also SW2.2
- net at BAR1.11 (K): no longer U1.40 (RB7/KBI3/PGD)
- net at BAR1.12 (K): no longer U1.39 (RB6/KBI2/PGC)
- net at BAR1.13 (K): now also U1.33 (RB0/AN12/INT0/FLT0/SDI/SDA); no longer U1.38 (RB5/KBI1/PGM)
- net at BAR1.14 (K): now also U1.34 (RB1/AN10/INT1/SCK/SCL); no longer U1.37 (RB4/AN11/KBI0/CSSPP)
- net at BAR1.15 (K): now also U1.35 (RB2/AN8/INT2/VMO); no longer U1.36 (RB3/AN9/CCP2/VPO)
- net at BAR1.16 (K): now also U1.36 (RB3/AN9/CCP2/VPO); no longer U1.35 (RB2/AN8/INT2/VMO)
- net at BAR1.17 (K): now also U1.37 (RB4/AN11/KBI0/CSSPP); no longer U1.34 (RB1/AN10/INT1/SCK/SCL)
- net at BAR1.18 (K): now also U1.38 (RB5/KBI1/PGM); no longer U1.33 (RB0/AN12/INT0/FLT0/SDI/SDA)
- net PGC: now reaches BAR1.19 (K)
- net PGC: now also U1.39 (RB6/KBI2/PGC)
- net PGD: now reaches BAR1.20 (K)
- net PGD: now also U1.40 (RB7/KBI3/PGD)
- net at U1.1 (Vpp/~{MCLR}/RE3): now also R19.1
- net MCLR-Debugger: now reaches SW2.1
- net MCLR-Debugger: now also R19.2, R20.1
- new net: R2.2, SW1.2, U1.14 (RA6/OSC2/CLKO)
- new net: R3.2, SW1.3, U1.7 (RA5/AN4/~{SS}/HLVDIN/C2OUT)
- new net: R4.2, SW1.4, U1.6 (RA4/T0CKI/C1OUT/RCV)
- new net: R5.2, SW1.5, U1.5 (RA3/AN3/Vref+)
- new net: R6.2, SW1.6, U1.4 (RA2/AN2/Vref-/CVref)
- new net: R7.2, SW1.7, U1.3 (RA1/AN1)
- new net: R8.2, SW1.8, U1.2 (RA0/AN0)
Other:
- added sheet LCD Display (lcd.kicad_sch)
- moved on the sheet: BAR1, R1, R9, SW1, SW2, U1

Commit message: Wiiiiiiiiiii
Other:
- added sheet Display 7 segmentos (untitled.kicad_sch)
- added sheet Dual display (untitled.kicad_sch)
Changed lines of the file:
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@@
+	)
+	(sheet
+		(at 464.82 7.62)
+		(size 151.13 116.84)
+		(exclude_from_sim no)
+		(in_bom yes)
+		(on_board yes)
+		(dnp no)
+		(fields_autoplaced yes)
+		(stroke
+			(width 0.1524)
+			(type solid)
+		)
+		(fill
+			(color 0 0 0 0.0000)
+		)
+		(property "Sheetname" "Display 7 segmentos"
+			(at 464.82 6.9084 0)
+			(effects
+				(font
+					(size 1.27 1.27)
+				)
+				(justify left bottom)
+			)
+		)
+		(property "Sheetfile" "untitled.kicad_sch"
+			(at 464.82 125.0446 0)
+			(effects
+				(font
+					(size 1.27 1.27)
+				)
+				(justify left top)
+			)
+		)
+		(instances
+			(project "Protoboard-Alejandra"
+				(path "/901f2ecb-0de8-4d14-a7e8-fe0a73fdd84c"
+					(page "3")
+				)
+			)
+		)
 	)
 	(sheet
@@
 				)
 			)
+		)
+	)
+	(sheet
+		(at 643.89 7.62)
+		(size 140.97 115.57)
+		(exclude_from_sim no)
+		(in_bom yes)
+		(on_board yes)
+		(dnp no)
+		(fields_autoplaced yes)
+		(stroke
+			(width 0.1524)
+			(type solid)
+		)
+		(fill
+			(color 0 0 0 0.0000)
+		)
+		(property "Sheetname" "Dual display"
+			(at 643.89 6.9084 0)
+			(effects
+				(font
+					(size 1.27 1.27)
+				)
+				(justify left bottom)
+			)
+		)
+		(property "Sheetfile" "untitled.kicad_sch"
+			(at 643.89 123.7746 0)
+			(effects
+				(font
+					(size 1.27 1.27)
+				)
+				(justify left top)
+			)
+		)
+		(instances
+			(project "Protoboard-Alejandra"
+				(path "/901f2ecb-0de8-4d14-a7e8-fe0a73fdd84c"
+					(page "4")
+				)
+			)
